File: kicad/motors.sch (KiCad schematic (older format))
At the start: 12 parts

Commit message: modified capacitors and cleaned up
Parts:
- removed C? (x2): 22u, symbol Device:CP1_Small
- removed C? (x2): C_Small, symbol Device:C_Small
- added C1, C4, C5, C8: 10u, symbol Device:CP_Small
- added D1, D10, D11, D12, D13, D2, D8, D9: D, symbol Device:D
- C2, C6: renamed from C?; value C_Small -> 0.1u
- C3, C7: renamed from C?; value 100n -> 0.1u
- J1: renamed from J?; value Conn_01x02 -> Left motor
- J4: renamed from J?; value Conn_01x02 -> Right motor
- gave numbers to parts that had none: 2
Connections:
- net +12V: now also C4.1, C8.1, D1.1 (K), D10.1 (K), D12.1 (K), D8.1 (K)
- net +3V3: now also C1.1, C5.1
- net GND: now also C1.2, C4.2, C5.2, C8.2, D11.2 (A), D13.2 (A), D2.2 (A), D9.2 (A)
- net M1_R: now also D1.2 (A), D10.2 (A), D11.1 (K), D2.1 (K)
- net ML_OUT2: now also D12.2 (A), D13.1 (K), D8.2 (A), D9.1 (K)
Other:
- note added: "EMF Protection"
- note added: "tutaj nie wiem czy elektrolit 10uF\nwystarczy na 12v, moze lepiej wiecej"
- moved on the sheet: C2, C3, U1

Commit message: modified capacitors near h bridge from 10u to 22u
Parts:
- C4, C8: value 10u -> 22u
Other:
- note removed: "tutaj nie wiem czy elektrolit 10uF\nwystarczy na 12v, moze lepiej wiecej"
Changed lines of the file:
@@
 P 4350 2850
 F 0 "C4" H 4438 2896 50  0000 L CNN
-F 1 "10u" H 4438 2805 50  0000 L CNN
+F 1 "22u" H 4438 2805 50  0000 L CNN
 F 2 "" H 4350 2850 50  0001 C CNN
 F 3 "~" H 4350 2850 50  0001 C CNN
@@
 P 8800 2850
 F 0 "C8" H 8888 2896 50  0000 L CNN
-F 1 "10u" H 8888 2805 50  0000 L CNN
+F 1 "22u" H 8888 2805 50  0000 L CNN
 F 2 "" H 8800 2850 50  0001 C CNN
 F 3 "~" H 8800 2850 50  0001 C CNN
@@
 $EndComp
 Connection ~ 8800 2950
-Text Notes 9050 2900 0    50   ~ 0
-tutaj nie wiem czy elektrolit 10uF\nwystarczy na 12v, moze lepiej wiecej
 $Comp
 L Device:D D10
@@
 	1    0    0    -1
 $EndComp
-Text Notes 4600 2900 0    50   ~ 0
-tutaj nie wiem czy elektrolit 10uF\nwystarczy na 12v, moze lepiej wiecej
 $Comp
 L power:GND #PWR0121

Commit message: fixed diodes, h bridge and modified power supply
Parts:
- added C? (x2): 500u, symbol Device:CP_Small
Connections:
- net +12V: now also C?.1, C?.1; no longer C4.1, C8.1
- net GND: now also C?.2, C?.2; no longer C4.2, C8.2
- net ML_OUT2: no longer D8.2 (A), D9.1 (K)
- net MR_OUT2: now also D8.2 (A), D9.1 (K)
Other:
- moved on the sheet: C4, C8
Changed lines of the file:
@@
 L Device:CP_Small C4
 U 1 1 60AF4E38
-P 4350 2850
-F 0 "C4" H 4438 2896 50  0000 L CNN
-F 1 "22u" H 4438 2805 50  0000 L CNN
-F 2 "" H 4350 2850 50  0001 C CNN
-F 3 "~" H 4350 2850 50  0001 C CNN
-	1    4350 2850
-	1    0    0    -1
-$EndComp
-Connection ~ 4350 2950
+P 4750 2850
+F 0 "C4" H 4838 2896 50  0000 L CNN
+F 1 "22u" H 4838 2805 50  0000 L CNN
+F 2 "" H 4750 2850 50  0001 C CNN
+F 3 "~" H 4750 2850 50  0001 C CNN
+	1    4750 2850
+	1    0    0    -1
+$EndComp
 $Comp
 L Device:CP_Small C5
@@
 L Device:CP_Small C8
 U 1 1 60AF7F2B
-P 8800 2850
-F 0 "C8" H 8888 2896 50  0000 L CNN
-F 1 "22u" H 8888 2805 50  0000 L CNN
-F 2 "" H 8800 2850 50  0001 C CNN
-F 3 "~" H 8800 2850 50  0001 C CNN
-	1    8800 2850
-	1    0    0    -1
-$EndComp
-Connection ~ 8800 2950
+P 9250 2850
+F 0 "C8" H 9338 2896 50  0000 L CNN
+F 1 "22u" H 9338 2805 50  0000 L CNN
+F 2 "" H 9250 2850 50  0001 C CNN
+F 3 "~" H 9250 2850 50  0001 C CNN
+	1    9250 2850
+	1    0    0    -1
+$EndComp
 $Comp
 L Device:D D10
@@
 	5300 4000 5300 4100
 Text GLabel 5000 4050 0    50   Input ~ 0
-ML_OUT1
+MR_OUT1
 Text GLabel 5300 4050 2    50   Input ~ 0
-ML_OUT2
+MR_OUT2
 Text Notes 9300 3400 0    50   ~ 0
 EMF Protection
@@
 	1    0    0    -1
 $EndComp
-Connection ~ 4350 2750
 $Comp
 L power:+12V #PWR0116
@@
 	1    0    0    -1
 $EndComp
-Connection ~ 8800 2750
 $Comp
 L power:+12V #PWR0119
@@
 	0    1    1    0
 $EndComp
+$Comp
+L Device:CP_Small C?
+U 1 1 60C28A06
+P 4350 2850
+F 0 "C?" H 4438 2896 50  0000 L CNN
+F 1 "500u" H 4438 2805 50  0000 L CNN
+F 2 "" H 4350 2850 50  0001 C CNN
+F 3 "~" H 4350 2850 50  0001 C CNN
+	1    4350 2850
+	1    0    0    -1
+$EndComp
+Connection ~ 4350 2750
+Connection ~ 4350 2950
+$Comp
+L Device:CP_Small C?
+U 1 1 60C2A88E
+P 8800 2850
+F 0 "C?" H 8888 2896 50  0000 L CNN
+F 1 "500u" H 8888 2805 50  0000 L CNN
+F 2 "" H 8800 2850 50  0001 C CNN
+F 3 "~" H 8800 2850 50  0001 C CNN
+	1    8800 2850
+	1    0    0    -1
+$EndComp
+Connection ~ 8800 2750
+Connection ~ 8800 2950
 $EndSCHEMATC

Commit message: deleted 3.3V and modified everything to use 5V instead
Parts:
- removed C4, C8: 22u, symbol Device:CP_Small
- J1, J4: footprint (none) -> Connector_PinSocket_2.54mm:PinSocket_1x02_P2.54mm_Vertical
- gave numbers to parts that had none: 2
Connections:
- net +3V3 renamed +5V
Changed lines of the file:
@@
 $EndComp
-Wire Wire Line
-	6550 2750 6700 2750
 Wire Wire Line
 	7150 3350 7150 2750
@@
 L_IN2
 $Comp
-L power:+3.3V #PWR?
-U 1 1 60B1D408
-P 6700 2750
-AR Path="/60B1D408" Ref="#PWR?"  Part="1"
-AR Path="/60AEE60B/60B1D408" Ref="#PWR0108"  Part="1"
-F 0 "#PWR0108" H 6700 2600 50  0001 C CNN
-F 1 "+3.3V" H 6715 2923 50  0000 C CNN
-F 2 "" H 6700 2750 50  0001 C CNN
-F 3 "" H 6700 2750 50  0001 C CNN
-	1    6700 2750
-	1    0    0    -1
-$EndComp
-Connection ~ 6700 2750
-Wire Wire Line
-	6700 2750 6850 2750
-$Comp
 L Connector_Generic:Conn_01x02 J1
 U 1 1 60B24363
@@
 F 0 "J1" H 10030 5792 50  0000 L CNN
 F 1 "Left motor" H 10030 5701 50  0000 L CNN
-F 2 "" H 9950 5800 50  0001 C CNN
+F 2 "Connector_PinSocket_2.54mm:PinSocket_1x02_P2.54mm_Vertical" H 9950 5800 50  0001 C CNN
 F 3 "~" H 9950 5800 50  0001 C CNN
 	1    9950 5800
@@
 F 0 "J4" H 10430 5792 50  0000 L CNN
 F 1 "Right motor" H 10430 5701 50  0000 L CNN
-F 2 "" H 10350 5800 50  0001 C CNN
+F 2 "Connector_PinSocket_2.54mm:PinSocket_1x02_P2.54mm_Vertical" H 10350 5800 50  0001 C CNN
 F 3 "~" H 10350 5800 50  0001 C CNN
 	1    10350 5800
@@
 $EndComp
 Wire Wire Line
-	2100 2750 2250 2750
-Wire Wire Line
 	2700 3350 2700 2750
 Wire Wire Line
@@
 Text GLabel 2700 4150 0    50   Input ~ 0
 R_IN2
-$Comp
-L power:+3.3V #PWR?
-U 1 1 60B481A2
-P 2250 2750
-AR Path="/60B481A2" Ref="#PWR?"  Part="1"
-AR Path="/60AEE60B/60B481A2" Ref="#PWR0112"  Part="1"
-F 0 "#PWR0112" H 2250 2600 50  0001 C CNN
-F 1 "+3.3V" H 2265 2923 50  0000 C CNN
-F 2 "" H 2250 2750 50  0001 C CNN
-F 3 "" H 2250 2750 50  0001 C CNN
-	1    2250 2750
-	1    0    0    -1
-$EndComp
-Connection ~ 2250 2750
-Wire Wire Line
-	2250 2750 2400 2750
 Wire Wire Line
 	3400 4750 3600 4750
@@
 $EndComp
 $Comp
-L Device:CP_Small C4
-U 1 1 60AF4E38
-P 4750 2850
-F 0 "C4" H 4838 2896 50  0000 L CNN
-F 1 "22u" H 4838 2805 50  0000 L CNN
-F 2 "" H 4750 2850 50  0001 C CNN
-F 3 "~" H 4750 2850 50  0001 C CNN
-	1    4750 2850
-	1    0    0    -1
-$EndComp
-$Comp
 L Device:CP_Small C5
 U 1 1 60AF6A3D
@@
 F 3 "~" H 6550 2850 50  0001 C CNN
 	1    6550 2850
-	1    0    0    -1
-$EndComp
-$Comp
-L Device:CP_Small C8
-U 1 1 60AF7F2B
-P 9250 2850
-F 0 "C8" H 9338 2896 50  0000 L CNN
-F 1 "22u" H 9338 2805 50  0000 L CNN
-F 2 "" H 9250 2850 50  0001 C CNN
-F 3 "~" H 9250 2850 50  0001 C CNN
-	1    9250 2850
 	1    0    0    -1
 $EndComp
@@
 $EndComp
 $Comp
-L Device:CP_Small C?
+L Device:CP_Small C4
 U 1 1 60C28A06
 P 4350 2850
-F 0 "C?" H 4438 2896 50  0000 L CNN
+F 0 "C4" H 4438 2896 50  0000 L CNN
 F 1 "500u" H 4438 2805 50  0000 L CNN
 F 2 "" H 4350 2850 50  0001 C CNN
@@
 Connection ~ 4350 2950
 $Comp
-L Device:CP_Small C?
+L Device:CP_Small C8
 U 1 1 60C2A88E
 P 8800 2850
-F 0 "C?" H 8888 2896 50  0000 L CNN
+F 0 "C8" H 8888 2896 50  0000 L CNN
 F 1 "500u" H 8888 2805 50  0000 L CNN
 F 2 "" H 8800 2850 50  0001 C CNN
@@
 Connection ~ 8800 2750
 Connection ~ 8800 2950
+Wire Wire Line
+	2100 2750 2250 2750
+$Comp
+L power:+5V #PWR0129
+U 1 1 60BDF66A
+P 2250 2750
+F 0 "#PWR0129" H 2250 2600 50  0001 C CNN
+F 1 "+5V" H 2265 2923 50  0000 C CNN
+F 2 "" H 2250 2750 50  0001 C CNN
+F 3 "" H 2250 2750 50  0001 C CNN
+	1    2250 2750
+	1    0    0    -1
+$EndComp
+Connection ~ 2250 2750
+Wire Wire Line
+	2250 2750 2400 2750
+Wire Wire Line
+	6550 2750 6700 2750
+$Comp
+L power:+5V #PWR0131
+U 1 1 60BE08B7
+P 6700 2750
+F 0 "#PWR0131" H 6700 2600 50  0001 C CNN
+F 1 "+5V" H 6715 2923 50  0000 C CNN
+F 2 "" H 6700 2750 50  0001 C CNN
+F 3 "" H 6700 2750 50  0001 C CNN
+	1    6700 2750
+	1    0    0    -1
+$EndComp
+Connection ~ 6700 2750
+Wire Wire Line
+	6700 2750 6850 2750
 $EndSCHEMATC

Commit message: created pcb view
Parts:
- C1, C5: footprint (none) -> Capacitor_THT:CP_Radial_D5.0mm_P2.00mm
- C2, C3, C6, C7: footprint (none) -> Capacitor_THT:C_Disc_D10.5mm_W5.0mm_P7.50mm
- C4, C8: value 500u -> 470u; footprint (none) -> Capacitor_THT:CP_Radial_D12.5mm_P5.00mm
- D1, D10, D11, D12, D13, D2, D8, D9: footprint (none) -> Diode_THT:D_DO-41_SOD81_P10.16mm_Horizontal
Changed lines of the file:
@@
 Text GLabel 8350 3350 2    0    Output ~ 0
 M1_R
-Text GLabel 8350 3550 2    50   Output ~ 0
+Text GLabel 8400 3550 2    50   Output ~ 0
 ML_OUT2
-Text GLabel 8350 3850 2    50   Output ~ 0
+Text GLabel 8400 3850 2    50   Output ~ 0
 ML_OUT1
-Text GLabel 8350 4050 2    50   Output ~ 0
+Text GLabel 8400 4050 2    50   Output ~ 0
 ML_OUT2
-Text GLabel 8350 3350 2    50   Output ~ 0
+Text GLabel 8400 3350 2    50   Output ~ 0
 ML_OUT1
 $Comp
@@
 F 0 "C7" H 8492 2896 50  0000 L CNN
 F 1 "0.1u" H 8492 2805 50  0000 L CNN
-F 2 "" H 8400 2850 50  0001 C CNN
+F 2 "Capacitor_THT:C_Disc_D10.5mm_W5.0mm_P7.50mm" H 8400 2850 50  0001 C CNN
 F 3 "~" H 8400 2850 50  0001 C CNN
 	1    8400 2850
@@
 F 0 "C6" H 6942 2896 50  0000 L CNN
 F 1 "0.1u" H 6942 2805 50  0000 L CNN
-F 2 "" H 6850 2850 50  0001 C CNN
+F 2 "Capacitor_THT:C_Disc_D10.5mm_W5.0mm_P7.50mm" H 6850 2850 50  0001 C CNN
 F 3 "~" H 6850 2850 50  0001 C CNN
 	1    6850 2850
@@
 Wire Wire Line
 	6700 2950 6850 2950
-Text GLabel 7150 3550 0    50   Input ~ 0
+Text GLabel 7100 3550 0    50   Input ~ 0
 PWM_L
-Text GLabel 7150 3850 0    50   Input ~ 0
+Text GLabel 7100 3850 0    50   Input ~ 0
 L_IN1
-Text GLabel 7150 3950 0    50   Input ~ 0
+Text GLabel 7100 3950 0    50   Input ~ 0
 L_IN2
-Text GLabel 7150 4050 0    50   Input ~ 0
+Text GLabel 7100 4050 0    50   Input ~ 0
 L_IN1
-Text GLabel 7150 4150 0    50   Input ~ 0
+Text GLabel 7100 4150 0    50   Input ~ 0
 L_IN2
 $Comp
@@
 Text GLabel 3900 3350 2    0    Output ~ 0
 M1_R
-Text GLabel 3900 3550 2    50   Output ~ 0
+Text GLabel 3950 3550 2    50   Output ~ 0
 MR_OUT2
-Text GLabel 3900 3850 2    50   Output ~ 0
+Text GLabel 3950 3850 2    50   Output ~ 0
 MR_OUT1
-Text GLabel 3900 4050 2    50   Output ~ 0
+Text GLabel 3950 4050 2    50   Output ~ 0
 MR_OUT2
-Text GLabel 3900 3350 2    50   Output ~ 0
+Text GLabel 3950 3350 2    50   Output ~ 0
 MR_OUT1
 $Comp
@@
 F 0 "C3" H 4042 2896 50  0000 L CNN
 F 1 "0.1u" H 4042 2805 50  0000 L CNN
-F 2 "" H 3950 2850 50  0001 C CNN
+F 2 "Capacitor_THT:C_Disc_D10.5mm_W5.0mm_P7.50mm" H 3950 2850 50  0001 C CNN
 F 3 "~" H 3950 2850 50  0001 C CNN
 	1    3950 2850
@@
 F 0 "C2" H 2492 2896 50  0000 L CNN
 F 1 "0.1u" H 2492 2805 50  0000 L CNN
-F 2 "" H 2400 2850 50  0001 C CNN
+F 2 "Capacitor_THT:C_Disc_D10.5mm_W5.0mm_P7.50mm" H 2400 2850 50  0001 C CNN
 F 3 "~" H 2400 2850 50  0001 C CNN
 	1    2400 2850
@@
 Wire Wire Line
 	2250 2950 2400 2950
-Text GLabel 2700 3550 0    50   Input ~ 0
+Text GLabel 2650 3550 0    50   Input ~ 0
 PWM_R
-Text GLabel 2700 3850 0    50   Input ~ 0
+Text GLabel 2650 3850 0    50   Input ~ 0
 R_IN1
-Text GLabel 2700 3950 0    50   Input ~ 0
+Text GLabel 2650 3950 0    50   Input ~ 0
 R_IN2
-Text GLabel 2700 4050 0    50   Input ~ 0
+Text GLabel 2650 4050 0    50   Input ~ 0
 R_IN1
-Text GLabel 2700 4150 0    50   Input ~ 0
+Text GLabel 2650 4150 0    50   Input ~ 0
 R_IN2
 Wire Wire Line
@@
 F 0 "C1" H 2188 2896 50  0000 L CNN
 F 1 "10u" H 2188 2805 50  0000 L CNN
-F 2 "" H 2100 2850 50  0001 C CNN
+F 2 "Capacitor_THT:CP_Radial_D5.0mm_P2.00mm" H 2100 2850 50  0001 C CNN
 F 3 "~" H 2100 2850 50  0001 C CNN
 	1    2100 2850
@@
 F 0 "C5" H 6638 2896 50  0000 L CNN
 F 1 "10u" H 6638 2805 50  0000 L CNN
-F 2 "" H 6550 2850 50  0001 C CNN
+F 2 "Capacitor_THT:CP_Radial_D5.0mm_P2.00mm" H 6550 2850 50  0001 C CNN
 F 3 "~" H 6550 2850 50  0001 C CNN
 	1    6550 2850
@@
 F 0 "D10" V 9354 3930 50  0000 L CNN
 F 1 "D" V 9445 3930 50  0000 L CNN
-F 2 "" H 9400 3850 50  0001 C CNN
+F 2 "Diode_THT:D_DO-41_SOD81_P10.16mm_Horizontal" H 9400 3850 50  0001 C CNN
 F 3 "~" H 9400 3850 50  0001 C CNN
 	1    9400 3850
@@
 F 0 "D11" V 9354 4330 50  0000 L CNN
 F 1 "D" V 9445 4330 50  0000 L CNN
-F 2 "" H 9400 4250 50  0001 C CNN
+F 2 "Diode_THT:D_DO-41_SOD81_P10.16mm_Horizontal" H 9400 4250 50  0001 C CNN
 F 3 "~" H 9400 4250 50  0001 C CNN
 	1    9400 4250
@@
 F 0 "D12" V 9654 3930 50  0000 L CNN
 F 1 "D" V 9745 3930 50  0000 L CNN
-F 2 "" H 9700 3850 50  0001 C CNN
+F 2 "Diode_THT:D_DO-41_SOD81_P10.16mm_Horizontal" H 9700 3850 50  0001 C CNN
 F 3 "~" H 9700 3850 50  0001 C CNN
 	1    9700 3850
@@
 F 0 "D13" V 9654 4330 50  0000 L CNN
 F 1 "D" V 9745 4330 50  0000 L CNN
-F 2 "" H 9700 4250 50  0001 C CNN
+F 2 "Diode_THT:D_DO-41_SOD81_P10.16mm_Horizontal" H 9700 4250 50  0001 C CNN
 F 3 "~" H 9700 4250 50  0001 C CNN
 	1    9700 4250
@@
 F 0 "D1" V 4954 3930 50  0000 L CNN
 F 1 "D" V 5045 3930 50  0000 L CNN
-F 2 "" H 5000 3850 50  0001 C CNN
+F 2 "Diode_THT:D_DO-41_SOD81_P10.16mm_Horizontal" H 5000 3850 50  0001 C CNN
 F 3 "~" H 5000 3850 50  0001 C CNN
 	1    5000 3850
@@
 $EndComp
 Wire Wire Line
-	5000 4000 5000 4100
+	5000 4000 5000 4050
 $Comp
 L Device:D D8
@@
 F 0 "D8" V 5254 3930 50  0000 L CNN
 F 1 "D" V 5345 3930 50  0000 L CNN
-F 2 "" H 5300 3850 50  0001 C CNN
+F 2 "Diode_THT:D_DO-41_SOD81_P10.16mm_Horizontal" H 5300 3850 50  0001 C CNN
 F 3 "~" H 5300 3850 50  0001 C CNN
 	1    5300 3850
@@
 $EndComp
 Wire Wire Line
-	5300 4000 5300 4100
-Text GLabel 5000 4050 0    50   Input ~ 0
+	5300 4000 5300 4050
+Text GLabel 4950 4050 0    50   Input ~ 0
 MR_OUT1
-Text GLabel 5300 4050 2    50   Input ~ 0
+Text GLabel 5350 4050 2    50   Input ~ 0
 MR_OUT2
 Text Notes 9300 3400 0    50   ~ 0
@@
 F 0 "D9" V 5254 4330 50  0000 L CNN
 F 1 "D" V 5345 4330 50  0000 L CNN
-F 2 "" H 5300 4250 50  0001 C CNN
+F 2 "Diode_THT:D_DO-41_SOD81_P10.16mm_Horizontal" H 5300 4250 50  0001 C CNN
 F 3 "~" H 5300 4250 50  0001 C CNN
 	1    5300 4250
@@
 F 0 "D2" V 4954 4330 50  0000 L CNN
 F 1 "D" V 5045 4330 50  0000 L CNN
-F 2 "" H 5000 4250 50  0001 C CNN
+F 2 "Diode_THT:D_DO-41_SOD81_P10.16mm_Horizontal" H 5000 4250 50  0001 C CNN
 F 3 "~" H 5000 4250 50  0001 C CNN
 	1    5000 4250
@@
 P 4350 2850
 F 0 "C4" H 4438 2896 50  0000 L CNN
-F 1 "500u" H 4438 2805 50  0000 L CNN
-F 2 "" H 4350 2850 50  0001 C CNN
+F 1 "470u" H 4438 2805 50  0000 L CNN
+F 2 "Capacitor_THT:CP_Radial_D12.5mm_P5.00mm" H 4350 2850 50  0001 C CNN
 F 3 "~" H 4350 2850 50  0001 C CNN
 	1    4350 2850
@@
 P 8800 2850
 F 0 "C8" H 8888 2896 50  0000 L CNN
-F 1 "500u" H 8888 2805 50  0000 L CNN
-F 2 "" H 8800 2850 50  0001 C CNN
+F 1 "470u" H 8888 2805 50  0000 L CNN
+F 2 "Capacitor_THT:CP_Radial_D12.5mm_P5.00mm" H 8800 2850 50  0001 C CNN
 F 3 "~" H 8800 2850 50  0001 C CNN
 	1    8800 2850
@@
 Wire Wire Line
 	6700 2750 6850 2750
+Wire Wire Line
+	3900 3350 3950 3350
+Wire Wire Line
+	3900 3550 3950 3550
+Wire Wire Line
+	3900 3850 3950 3850
+Wire Wire Line
+	3900 4050 3950 4050
+Wire Wire Line
+	2700 4150 2650 4150
+Wire Wire Line
+	2700 4050 2650 4050
+Wire Wire Line
+	2700 3950 2650 3950
+Wire Wire Line
+	2700 3850 2650 3850
+Wire Wire Line
+	2650 3550 2700 3550
+Connection ~ 2700 3550
+Wire Wire Line
+	7100 3550 7150 3550
+Connection ~ 7150 3550
+Wire Wire Line
+	7100 3850 7150 3850
+Wire Wire Line
+	7100 3950 7150 3950
+Wire Wire Line
+	7100 4050 7150 4050
+Wire Wire Line
+	7100 4150 7150 4150
+Wire Wire Line
+	8350 3350 8400 3350
+Wire Wire Line
+	8350 3550 8400 3550
+Wire Wire Line
+	8350 3850 8400 3850
+Wire Wire Line
+	8350 4050 8400 4050
+Wire Wire Line
+	4950 4050 5000 4050
+Connection ~ 5000 4050
+Wire Wire Line
+	5000 4050 5000 4100
+Wire Wire Line
+	5350 4050 5300 4050
+Connection ~ 5300 4050
+Wire Wire Line
+	5300 4050 5300 4100
 $EndSCHEMATC
