File: kicad/power.sch (KiCad schematic (older format))
At the start: 17 parts, among them J5 Li-Po balancer, SW1 SW_SPDT, SW2 SW_SPDT, U3 LM1117-5.0, U4 LM1117-3.3

Commit message: fixed diodes, h bridge and modified power supply
Parts:
- removed D15: LED, symbol Device:LED
- removed R2: 1000, symbol Device:R
- removed SW1: SW_SPDT, symbol Switch:SW_SPDT
- added C?: 0.1u, symbol Device:C_Small
- added R?: 220k, symbol Device:R_Small
- added R?: 82k, symbol Device:R_Small
- R1: value 500 -> 1k
Connections:
- net +8V is gone; now on net +12V: C11.1, C9.1, U3.3 (VI)
- net +12V: now also R?.2
- net GND: now also C?.1, R?.2
- new net BAT_PROBE: C?.2, R?.1, R?.1
Other:
- note added: "Battery probe"
- note added: "Vmax = 12,6 V\nR1 = 220 kOhm\nR2 = 82 kOhm\nVout = 3,421 V -> mniej niż zakres ADC (3,6V)\nI = 12,6 / 302k = 41uA -> malutko czyli bateria nie będzie się mocno rozładowywać"
- moved on the sheet: D14, R1, SW2
Changed lines of the file:
@@
-$Comp
-L Switch:SW_SPDT SW?
-U 1 1 60B5B7C0
-P 3050 4700
-AR Path="/60B5B7C0" Ref="SW?"  Part="1"
-AR Path="/60AFA27C/60B5B7C0" Ref="SW1"  Part="1"
-F 0 "SW1" H 3050 4985 50  0000 C CNN
-F 1 "SW_SPDT" H 3050 4894 50  0000 C CNN
-F 2 "" H 3050 4700 50  0001 C CNN
-F 3 "~" H 3050 4700 50  0001 C CNN
-	1    3050 4700
-	0    1    1    0
-$EndComp
-Wire Wire Line
-	3300 3800 3300 4500
-Wire Wire Line
-	3300 4500 3050 4500
-NoConn ~ 3150 4900
-Wire Wire Line
-	3400 3800 3400 4500
-Wire Wire Line
-	3400 4500 3500 4500
 $Comp
 L Switch:SW_SPDT SW?
 U 1 1 60B5B7CC
-P 3500 4700
+P 3400 4050
 AR Path="/60B5B7CC" Ref="SW?"  Part="1"
 AR Path="/60AFA27C/60B5B7CC" Ref="SW2"  Part="1"
-F 0 "SW2" H 3500 4985 50  0000 C CNN
-F 1 "SW_SPDT" H 3500 4894 50  0000 C CNN
-F 2 "" H 3500 4700 50  0001 C CNN
-F 3 "~" H 3500 4700 50  0001 C CNN
-	1    3500 4700
-	0    1    1    0
-$EndComp
-NoConn ~ 3600 4900
-$Comp
-L Device:R R?
-U 1 1 60B5B7D4
-P 4350 4300
-AR Path="/60B5B7D4" Ref="R?"  Part="1"
-AR Path="/60AFA27C/60B5B7D4" Ref="R2"  Part="1"
-F 0 "R2" H 4420 4346 50  0000 L CNN
-F 1 "1000" H 4420 4255 50  0000 L CNN
-F 2 "" V 4280 4300 50  0001 C CNN
-F 3 "~" H 4350 4300 50  0001 C CNN
-	1    4350 4300
-	-1   0    0    1
-$EndComp
+F 0 "SW2" H 3400 4335 50  0000 C CNN
+F 1 "SW_SPDT" H 3400 4244 50  0000 C CNN
+F 2 "" H 3400 4050 50  0001 C CNN
+F 3 "~" H 3400 4050 50  0001 C CNN
+	1    3400 4050
+	0    1    1    0
+$EndComp
+NoConn ~ 3500 4250
 $Comp
 L Device:R R?
 U 1 1 60B5B7DA
-P 3950 4300
+P 4200 4300
 AR Path="/60B5B7DA" Ref="R?"  Part="1"
 AR Path="/60AFA27C/60B5B7DA" Ref="R1"  Part="1"
-F 0 "R1" H 4020 4346 50  0000 L CNN
-F 1 "500" H 4020 4255 50  0000 L CNN
-F 2 "" V 3880 4300 50  0001 C CNN
-F 3 "~" H 3950 4300 50  0001 C CNN
-	1    3950 4300
-	-1   0    0    1
-$EndComp
-$Comp
-L Device:LED D?
-U 1 1 60B5B7E0
-P 4350 4000
-AR Path="/60B5B7E0" Ref="D?"  Part="1"
-AR Path="/60AFA27C/60B5B7E0" Ref="D15"  Part="1"
-F 0 "D15" V 4389 3882 50  0000 R CNN
-F 1 "LED" V 4298 3882 50  0000 R CNN
-F 2 "" H 4350 4000 50  0001 C CNN
-F 3 "~" H 4350 4000 50  0001 C CNN
-	1    4350 4000
-	0    1    1    0
+F 0 "R1" H 4270 4346 50  0000 L CNN
+F 1 "1k" H 4270 4255 50  0000 L CNN
+F 2 "" V 4130 4300 50  0001 C CNN
+F 3 "~" H 4200 4300 50  0001 C CNN
+	1    4200 4300
+	-1   0    0    1
 $EndComp
 $Comp
 L Device:LED D?
 U 1 1 60B5B7E6
-P 3950 4000
+P 4200 4000
 AR Path="/60B5B7E6" Ref="D?"  Part="1"
 AR Path="/60AFA27C/60B5B7E6" Ref="D14"  Part="1"
-F 0 "D14" V 3989 3882 50  0000 R CNN
-F 1 "LED" V 3898 3882 50  0000 R CNN
-F 2 "" H 3950 4000 50  0001 C CNN
-F 3 "~" H 3950 4000 50  0001 C CNN
-	1    3950 4000
+F 0 "D14" V 4239 3882 50  0000 R CNN
+F 1 "LED" V 4148 3882 50  0000 R CNN
+F 2 "" H 4200 4000 50  0001 C CNN
+F 3 "~" H 4200 4000 50  0001 C CNN
+	1    4200 4000
 	0    1    1    0
 $EndComp
@@
 L power:GND #PWR?
 U 1 1 60B5B7EC
-P 4150 3700
+P 4200 3700
 AR Path="/60B5B7EC" Ref="#PWR?"  Part="1"
 AR Path="/60AFA27C/60B5B7EC" Ref="#PWR0127"  Part="1"
-F 0 "#PWR0127" H 4150 3450 50  0001 C CNN
-F 1 "GND" H 4155 3527 50  0000 C CNN
-F 2 "" H 4150 3700 50  0001 C CNN
-F 3 "" H 4150 3700 50  0001 C CNN
-	1    4150 3700
-	-1   0    0    1
-$EndComp
-Wire Wire Line
-	4350 3850 4350 3700
-Wire Wire Line
-	3950 3850 3950 3700
-Wire Wire Line
-	4350 3700 4150 3700
-Wire Wire Line
-	4150 3700 3950 3700
-Connection ~ 4150 3700
+F 0 "#PWR0127" H 4200 3450 50  0001 C CNN
+F 1 "GND" H 4205 3527 50  0000 C CNN
+F 2 "" H 4200 3700 50  0001 C CNN
+F 3 "" H 4200 3700 50  0001 C CNN
+	1    4200 3700
+	-1   0    0    1
+$EndComp
+Wire Wire Line
+	4200 3850 4200 3700
 $Comp
 L power:+12V #PWR0128
 U 1 1 60B7695D
-P 3400 4900
-F 0 "#PWR0128" H 3400 4750 50  0001 C CNN
-F 1 "+12V" H 3415 5073 50  0000 C CNN
-F 2 "" H 3400 4900 50  0001 C CNN
-F 3 "" H 3400 4900 50  0001 C CNN
-	1    3400 4900
-	-1   0    0    1
-$EndComp
-$Comp
-L power:+8V #PWR0129
-U 1 1 60B77613
-P 2950 4900
-F 0 "#PWR0129" H 2950 4750 50  0001 C CNN
-F 1 "+8V" H 2965 5073 50  0000 C CNN
-F 2 "" H 2950 4900 50  0001 C CNN
-F 3 "" H 2950 4900 50  0001 C CNN
-	1    2950 4900
+P 3300 4250
+F 0 "#PWR0128" H 3300 4100 50  0001 C CNN
+F 1 "+12V" H 3315 4423 50  0000 C CNN
+F 2 "" H 3300 4250 50  0001 C CNN
+F 3 "" H 3300 4250 50  0001 C CNN
+	1    3300 4250
 	-1   0    0    1
 $EndComp
@@
 L power:+12V #PWR0130
 U 1 1 60B7851F
-P 3950 4450
-F 0 "#PWR0130" H 3950 4300 50  0001 C CNN
-F 1 "+12V" H 3965 4623 50  0000 C CNN
-F 2 "" H 3950 4450 50  0001 C CNN
-F 3 "" H 3950 4450 50  0001 C CNN
-	1    3950 4450
-	-1   0    0    1
-$EndComp
-$Comp
-L power:+8V #PWR0131
-U 1 1 60B78FB3
-P 4350 4450
-F 0 "#PWR0131" H 4350 4300 50  0001 C CNN
-F 1 "+8V" H 4365 4623 50  0000 C CNN
-F 2 "" H 4350 4450 50  0001 C CNN
-F 3 "" H 4350 4450 50  0001 C CNN
-	1    4350 4450
-	-1   0    0    1
-$EndComp
-$Comp
-L power:+8V #PWR0132
-U 1 1 60B7B402
-P 5250 4100
-F 0 "#PWR0132" H 5250 3950 50  0001 C CNN
-F 1 "+8V" H 5265 4273 50  0000 C CNN
-F 2 "" H 5250 4100 50  0001 C CNN
-F 3 "" H 5250 4100 50  0001 C CNN
-	1    5250 4100
-	1    0    0    -1
-$EndComp
-Connection ~ 5250 4100
+P 4200 4450
+F 0 "#PWR0130" H 4200 4300 50  0001 C CNN
+F 1 "+12V" H 4215 4623 50  0000 C CNN
+F 2 "" H 4200 4450 50  0001 C CNN
+F 3 "" H 4200 4450 50  0001 C CNN
+	1    4200 4450
+	-1   0    0    1
+$EndComp
 $Comp
 L power:+5V #PWR0133
@@
 $EndComp
 Connection ~ 7350 4100
+NoConn ~ 3300 3800
+Wire Wire Line
+	3400 3800 3400 3850
+$Comp
+L power:+12V #PWR?
+U 1 1 60BD6F1B
+P 5250 4100
+F 0 "#PWR?" H 5250 3950 50  0001 C CNN
+F 1 "+12V" H 5265 4273 50  0000 C CNN
+F 2 "" H 5250 4100 50  0001 C CNN
+F 3 "" H 5250 4100 50  0001 C CNN
+	1    5250 4100
+	1    0    0    -1
+$EndComp
+Connection ~ 5250 4100
+Text Notes 1750 5700 0    79   ~ 0
+Battery probe
+$Comp
+L power:+12V #PWR?
+U 1 1 60C15EFB
+P 1500 6000
+F 0 "#PWR?" H 1500 5850 50  0001 C CNN
+F 1 "+12V" V 1515 6128 50  0000 L CNN
+F 2 "" H 1500 6000 50  0001 C CNN
+F 3 "" H 1500 6000 50  0001 C CNN
+	1    1500 6000
+	0    -1   -1   0
+$EndComp
+$Comp
+L power:GND #PWR?
+U 1 1 60C16CCC
+P 2650 6000
+F 0 "#PWR?" H 2650 5750 50  0001 C CNN
+F 1 "GND" V 2655 5872 50  0000 R CNN
+F 2 "" H 2650 6000 50  0001 C CNN
+F 3 "" H 2650 6000 50  0001 C CNN
+	1    2650 6000
+	0    -1   -1   0
+$EndComp
+$Comp
+L Device:R_Small R?
+U 1 1 60C18049
+P 1800 6000
+F 0 "R?" V 1604 6000 50  0000 C CNN
+F 1 "220k" V 1695 6000 50  0000 C CNN
+F 2 "" H 1800 6000 50  0001 C CNN
+F 3 "~" H 1800 6000 50  0001 C CNN
+	1    1800 6000
+	0    1    1    0
+$EndComp
+$Comp
+L Device:R_Small R?
+U 1 1 60C18CC7
+P 2400 6000
+F 0 "R?" V 2596 6000 50  0000 C CNN
+F 1 "82k" V 2505 6000 50  0000 C CNN
+F 2 "" H 2400 6000 50  0001 C CNN
+F 3 "~" H 2400 6000 50  0001 C CNN
+	1    2400 6000
+	0    -1   -1   0
+$EndComp
+Wire Wire Line
+	1500 6000 1700 6000
+Wire Wire Line
+	1900 6000 2100 6000
+Wire Wire Line
+	2500 6000 2600 6000
+$Comp
+L Device:C_Small C?
+U 1 1 60C1A620
+P 2400 6350
+F 0 "C?" V 2171 6350 50  0000 C CNN
+F 1 "0.1u" V 2262 6350 50  0000 C CNN
+F 2 "" H 2400 6350 50  0001 C CNN
+F 3 "~" H 2400 6350 50  0001 C CNN
+	1    2400 6350
+	0    1    1    0
+$EndComp
+Wire Wire Line
+	2500 6350 2600 6350
+Wire Wire Line
+	2600 6350 2600 6000
+Connection ~ 2600 6000
+Wire Wire Line
+	2600 6000 2650 6000
+Text Notes 3050 6100 0    39   ~ 0
+Vmax = 12,6 V\nR1 = 220 kOhm\nR2 = 82 kOhm\nVout = 3,421 V -> mniej niż zakres ADC (3,6V)\nI = 12,6 / 302k = 41uA -> malutko czyli bateria nie będzie się mocno rozładowywać
+Text GLabel 2000 6250 0    50   Output ~ 0
+BAT_PROBE
+Wire Wire Line
+	2300 6350 2100 6350
+Wire Wire Line
+	2100 6350 2100 6250
+Connection ~ 2100 6000
+Wire Wire Line
+	2100 6000 2300 6000
+Wire Wire Line
+	2000 6250 2100 6250
+Connection ~ 2100 6250
+Wire Wire Line
+	2100 6250 2100 6000
 $EndSCHEMATC

Commit message: deleted 3.3V and modified everything to use 5V instead
Parts:
- removed C15, C18: 0.1u, symbol Device:C_Small
- removed C16, C17: 10u, symbol Device:CP_Small
- removed U4: LM1117-3.3, symbol Regulator_Linear:LM1117-3.3
- D14: footprint (none) -> LED_THT:LED_D5.0mm
- J5: footprint (none) -> Connector_JST:JST_XH_B4B-XH-A_1x04_P2.50mm_Vertical
- gave numbers to parts that had none: 3
Other:
- note removed: "3.3V Power regulator"
Changed lines of the file:
@@
 	6400 4100 6500 4100
 Connection ~ 6500 4100
-$Comp
-L Regulator_Linear:LM1117-3.3 U?
-U 1 1 60B46B9E
-P 8200 4100
-AR Path="/60B46B9E" Ref="U?"  Part="1"
-AR Path="/60AFA27C/60B46B9E" Ref="U4"  Part="1"
-F 0 "U4" H 8200 4342 50  0000 C CNN
-F 1 "LM1117-3.3" H 8200 4251 50  0000 C CNN
-F 2 "" H 8200 4100 50  0001 C CNN
-F 3 "http://www.ti.com/lit/ds/symlink/lm1117.pdf" H 8200 4100 50  0001 C CNN
-	1    8200 4100
-	1    0    0    -1
-$EndComp
 Wire Wire Line
 	5250 4400 5650 4400
@@
 Wire Wire Line
 	5650 4400 6100 4400
-$Comp
-L Device:C_Small C?
-U 1 1 60B46BAB
-P 7350 4200
-AR Path="/60B46BAB" Ref="C?"  Part="1"
-AR Path="/60AFA27C/60B46BAB" Ref="C15"  Part="1"
-F 0 "C15" H 7442 4246 50  0000 L CNN
-F 1 "0.1u" H 7442 4155 50  0000 L CNN
-F 2 "" H 7350 4200 50  0001 C CNN
-F 3 "~" H 7350 4200 50  0001 C CNN
-	1    7350 4200
-	1    0    0    -1
-$EndComp
-$Comp
-L Device:CP_Small C?
-U 1 1 60B46BB1
-P 7750 4200
-AR Path="/60B46BB1" Ref="C?"  Part="1"
-AR Path="/60AFA27C/60B46BB1" Ref="C16"  Part="1"
-F 0 "C16" H 7838 4246 50  0000 L CNN
-F 1 "10u" H 7838 4155 50  0000 L CNN
-F 2 "" H 7750 4200 50  0001 C CNN
-F 3 "~" H 7750 4200 50  0001 C CNN
-	1    7750 4200
-	1    0    0    -1
-$EndComp
-$Comp
-L Device:CP_Small C?
-U 1 1 60B46BB7
-P 8600 4200
-AR Path="/60B46BB7" Ref="C?"  Part="1"
-AR Path="/60AFA27C/60B46BB7" Ref="C17"  Part="1"
-F 0 "C17" H 8688 4246 50  0000 L CNN
-F 1 "10u" H 8688 4155 50  0000 L CNN
-F 2 "" H 8600 4200 50  0001 C CNN
-F 3 "~" H 8600 4200 50  0001 C CNN
-	1    8600 4200
-	1    0    0    -1
-$EndComp
-$Comp
-L Device:C_Small C?
-U 1 1 60B46BBD
-P 8900 4200
-AR Path="/60B46BBD" Ref="C?"  Part="1"
-AR Path="/60AFA27C/60B46BBD" Ref="C18"  Part="1"
-F 0 "C18" H 8992 4246 50  0000 L CNN
-F 1 "0.1u" H 8992 4155 50  0000 L CNN
-F 2 "" H 8900 4200 50  0001 C CNN
-F 3 "~" H 8900 4200 50  0001 C CNN
-	1    8900 4200
-	1    0    0    -1
-$EndComp
-Wire Wire Line
-	7350 4300 7350 4400
-Wire Wire Line
-	8600 4400 8600 4300
-Wire Wire Line
-	8600 4100 8900 4100
-Wire Wire Line
-	8900 4300 8900 4400
-Wire Wire Line
-	8900 4400 8600 4400
-Connection ~ 8600 4400
-$Comp
-L power:GND #PWR?
-U 1 1 60B46BC9
-P 8900 4400
-AR Path="/60B46BC9" Ref="#PWR?"  Part="1"
-AR Path="/60AFA27C/60B46BC9" Ref="#PWR0124"  Part="1"
-F 0 "#PWR0124" H 8900 4150 50  0001 C CNN
-F 1 "GND" H 8905 4227 50  0000 C CNN
-F 2 "" H 8900 4400 50  0001 C CNN
-F 3 "" H 8900 4400 50  0001 C CNN
-	1    8900 4400
-	1    0    0    -1
-$EndComp
-Connection ~ 8900 4400
-Wire Wire Line
-	8500 4100 8600 4100
-Connection ~ 8600 4100
-Wire Wire Line
-	7350 4400 7750 4400
-Wire Wire Line
-	7350 4100 7750 4100
-Connection ~ 7750 4100
-Wire Wire Line
-	7750 4300 7750 4400
-Wire Wire Line
-	7750 4100 7900 4100
-Connection ~ 7750 4400
-Wire Wire Line
-	7750 4400 8200 4400
-Connection ~ 8200 4400
-Wire Wire Line
-	8200 4400 8600 4400
-$Comp
-L power:+3.3V #PWR?
-U 1 1 60B46BDD
-P 8900 4100
-AR Path="/60B46BDD" Ref="#PWR?"  Part="1"
-AR Path="/60AFA27C/60B46BDD" Ref="#PWR0125"  Part="1"
-F 0 "#PWR0125" H 8900 3950 50  0001 C CNN
-F 1 "+3.3V" H 8915 4273 50  0000 C CNN
-F 2 "" H 8900 4100 50  0001 C CNN
-F 3 "" H 8900 4100 50  0001 C CNN
-	1    8900 4100
-	1    0    0    -1
-$EndComp
-Connection ~ 8900 4100
-Text Notes 7550 3700 0    79   ~ 0
-3.3V Power regulator
 $Comp
 L Connector_Generic:Conn_01x04 J?
@@
 F 0 "J5" H 3118 3175 50  0000 C CNN
 F 1 "Li-Po balancer" H 3118 3266 50  0000 C CNN
-F 2 "" H 3200 3600 50  0001 C CNN
+F 2 "Connector_JST:JST_XH_B4B-XH-A_1x04_P2.50mm_Vertical" H 3200 3600 50  0001 C CNN
 F 3 "~" H 3200 3600 50  0001 C CNN
 	1    3200 3600
@@
 F 0 "D14" V 4239 3882 50  0000 R CNN
 F 1 "LED" V 4148 3882 50  0000 R CNN
-F 2 "" H 4200 4000 50  0001 C CNN
+F 2 "LED_THT:LED_D5.0mm" H 4200 4000 50  0001 C CNN
 F 3 "~" H 4200 4000 50  0001 C CNN
 	1    4200 4000
@@
 $EndComp
 Connection ~ 6800 4100
-$Comp
-L power:+5V #PWR0134
-U 1 1 60B7CE96
-P 7350 4100
-F 0 "#PWR0134" H 7350 3950 50  0001 C CNN
-F 1 "+5V" H 7365 4273 50  0000 C CNN
-F 2 "" H 7350 4100 50  0001 C CNN
-F 3 "" H 7350 4100 50  0001 C CNN
-	1    7350 4100
-	1    0    0    -1
-$EndComp
-Connection ~ 7350 4100
 NoConn ~ 3300 3800
 Wire Wire Line
 	3400 3800 3400 3850
 $Comp
-L power:+12V #PWR?
+L power:+12V #PWR0132
 U 1 1 60BD6F1B
 P 5250 4100
-F 0 "#PWR?" H 5250 3950 50  0001 C CNN
+F 0 "#PWR0132" H 5250 3950 50  0001 C CNN
 F 1 "+12V" H 5265 4273 50  0000 C CNN
 F 2 "" H 5250 4100 50  0001 C CNN
@@
 Battery probe
 $Comp
-L power:+12V #PWR?
+L power:+12V #PWR0134
 U 1 1 60C15EFB
 P 1500 6000
-F 0 "#PWR?" H 1500 5850 50  0001 C CNN
+F 0 "#PWR0134" H 1500 5850 50  0001 C CNN
 F 1 "+12V" V 1515 6128 50  0000 L CNN
 F 2 "" H 1500 6000 50  0001 C CNN
@@
 $EndComp
 $Comp
-L power:GND #PWR?
+L power:GND #PWR0143
 U 1 1 60C16CCC
 P 2650 6000
-F 0 "#PWR?" H 2650 5750 50  0001 C CNN
+F 0 "#PWR0143" H 2650 5750 50  0001 C CNN
 F 1 "GND" V 2655 5872 50  0000 R CNN
 F 2 "" H 2650 6000 50  0001 C CNN
@@
 $EndComp
 $Comp
-L Device:R_Small R?
+L Device:R_Small R2
 U 1 1 60C18049
 P 1800 6000
-F 0 "R?" V 1604 6000 50  0000 C CNN
+F 0 "R2" V 1604 6000 50  0000 C CNN
 F 1 "220k" V 1695 6000 50  0000 C CNN
 F 2 "" H 1800 6000 50  0001 C CNN
@@
 $EndComp
 $Comp
-L Device:R_Small R?
+L Device:R_Small R18
 U 1 1 60C18CC7
 P 2400 6000
-F 0 "R?" V 2596 6000 50  0000 C CNN
+F 0 "R18" V 2596 6000 50  0000 C CNN
 F 1 "82k" V 2505 6000 50  0000 C CNN
 F 2 "" H 2400 6000 50  0001 C CNN
@@
 	2500 6000 2600 6000
 $Comp
-L Device:C_Small C?
+L Device:C_Small C15
 U 1 1 60C1A620
 P 2400 6350
-F 0 "C?" V 2171 6350 50  0000 C CNN
+F 0 "C15" V 2171 6350 50  0000 C CNN
 F 1 "0.1u" V 2262 6350 50  0000 C CNN
 F 2 "" H 2400 6350 50  0001 C CNN

Commit message: created pcb view
Parts:
- C11, C13: footprint (none) -> Capacitor_THT:CP_Radial_D5.0mm_P2.00mm
- C14, C15, C9: footprint (none) -> Capacitor_THT:C_Disc_D10.5mm_W5.0mm_P7.50mm
- R1: footprint (none) -> Resistor_SMD:R_1206_3216Metric_Pad1.30x1.75mm_HandSolder
- R18: value 82k -> 75k; footprint (none) -> Resistor_SMD:R_1206_3216Metric_Pad1.30x1.75mm_HandSolder
- R2: value 220k -> 200k; footprint (none) -> Resistor_SMD:R_1206_3216Metric_Pad1.30x1.75mm_HandSolder
- SW2: footprint (none) -> Button_Switch_THT:SW_Push_1P2T_Vertical_E-Switch_800UDP8P1A1M6
- U3: footprint (none) -> warsztaty:LM1117_TO-252
Other:
- note added: "Vmax = 12,6 V\nR1 = 200 kOhm\nR2 = 75 kOhm\nVout = 3,436 V -> mniej niż zakres ADC (3,6V)\nI = 12,6 / 275k = 45uA -> malutko czyli bateria nie będzie się mocno rozładowywać"
- note removed: "Vmax = 12,6 V\nR1 = 220 kOhm\nR2 = 82 kOhm\nVout = 3,421 V -> mniej niż zakres ADC (3,6V)\nI = 12,6 / 302k = 41uA -> malutko czyli bateria nie będzie się mocno rozładowywać"
Changed lines of the file:
@@
 F 0 "C9" H 5342 4246 50  0000 L CNN
 F 1 "0.1u" H 5342 4155 50  0000 L CNN
-F 2 "" H 5250 4200 50  0001 C CNN
+F 2 "Capacitor_THT:C_Disc_D10.5mm_W5.0mm_P7.50mm" H 5250 4200 50  0001 C CNN
 F 3 "~" H 5250 4200 50  0001 C CNN
 	1    5250 4200
@@
 F 0 "C11" H 5738 4246 50  0000 L CNN
 F 1 "10u" H 5738 4155 50  0000 L CNN
-F 2 "" H 5650 4200 50  0001 C CNN
+F 2 "Capacitor_THT:CP_Radial_D5.0mm_P2.00mm" H 5650 4200 50  0001 C CNN
 F 3 "~" H 5650 4200 50  0001 C CNN
 	1    5650 4200
@@
 F 0 "C13" H 6588 4246 50  0000 L CNN
 F 1 "10u" H 6588 4155 50  0000 L CNN
-F 2 "" H 6500 4200 50  0001 C CNN
+F 2 "Capacitor_THT:CP_Radial_D5.0mm_P2.00mm" H 6500 4200 50  0001 C CNN
 F 3 "~" H 6500 4200 50  0001 C CNN
 	1    6500 4200
@@
 F 0 "C14" H 6892 4246 50  0000 L CNN
 F 1 "0.1u" H 6892 4155 50  0000 L CNN
-F 2 "" H 6800 4200 50  0001 C CNN
+F 2 "Capacitor_THT:C_Disc_D10.5mm_W5.0mm_P7.50mm" H 6800 4200 50  0001 C CNN
 F 3 "~" H 6800 4200 50  0001 C CNN
 	1    6800 4200
@@
 F 0 "U3" H 6100 4342 50  0000 C CNN
 F 1 "LM1117-5.0" H 6100 4251 50  0000 C CNN
-F 2 "" H 6100 4100 50  0001 C CNN
+F 2 "warsztaty:LM1117_TO-252" H 6100 4100 50  0001 C CNN
 F 3 "http://www.ti.com/lit/ds/symlink/lm1117.pdf" H 6100 4100 50  0001 C CNN
 	1    6100 4100
@@
 F 0 "SW2" H 3400 4335 50  0000 C CNN
 F 1 "SW_SPDT" H 3400 4244 50  0000 C CNN
-F 2 "" H 3400 4050 50  0001 C CNN
+F 2 "Button_Switch_THT:SW_Push_1P2T_Vertical_E-Switch_800UDP8P1A1M6" H 3400 4050 50  0001 C CNN
 F 3 "~" H 3400 4050 50  0001 C CNN
 	1    3400 4050
@@
 F 0 "R1" H 4270 4346 50  0000 L CNN
 F 1 "1k" H 4270 4255 50  0000 L CNN
-F 2 "" V 4130 4300 50  0001 C CNN
+F 2 "Resistor_SMD:R_1206_3216Metric_Pad1.30x1.75mm_HandSolder" V 4130 4300 50  0001 C CNN
 F 3 "~" H 4200 4300 50  0001 C CNN
 	1    4200 4300
@@
 P 1800 6000
 F 0 "R2" V 1604 6000 50  0000 C CNN
-F 1 "220k" V 1695 6000 50  0000 C CNN
-F 2 "" H 1800 6000 50  0001 C CNN
+F 1 "200k" V 1695 6000 50  0000 C CNN
+F 2 "Resistor_SMD:R_1206_3216Metric_Pad1.30x1.75mm_HandSolder" H 1800 6000 50  0001 C CNN
 F 3 "~" H 1800 6000 50  0001 C CNN
 	1    1800 6000
@@
 P 2400 6000
 F 0 "R18" V 2596 6000 50  0000 C CNN
-F 1 "82k" V 2505 6000 50  0000 C CNN
-F 2 "" H 2400 6000 50  0001 C CNN
+F 1 "75k" V 2505 6000 50  0000 C CNN
+F 2 "Resistor_SMD:R_1206_3216Metric_Pad1.30x1.75mm_HandSolder" H 2400 6000 50  0001 C CNN
 F 3 "~" H 2400 6000 50  0001 C CNN
 	1    2400 6000
@@
 F 0 "C15" V 2171 6350 50  0000 C CNN
 F 1 "0.1u" V 2262 6350 50  0000 C CNN
-F 2 "" H 2400 6350 50  0001 C CNN
+F 2 "Capacitor_THT:C_Disc_D10.5mm_W5.0mm_P7.50mm" H 2400 6350 50  0001 C CNN
 F 3 "~" H 2400 6350 50  0001 C CNN
 	1    2400 6350
@@
 	2600 6000 2650 6000
 Text Notes 3050 6100 0    39   ~ 0
-Vmax = 12,6 V\nR1 = 220 kOhm\nR2 = 82 kOhm\nVout = 3,421 V -> mniej niż zakres ADC (3,6V)\nI = 12,6 / 302k = 41uA -> malutko czyli bateria nie będzie się mocno rozładowywać
+Vmax = 12,6 V\nR1 = 200 kOhm\nR2 = 75 kOhm\nVout = 3,436 V -> mniej niż zakres ADC (3,6V)\nI = 12,6 / 275k = 45uA -> malutko czyli bateria nie będzie się mocno rozładowywać
 Text GLabel 2000 6250 0    50   Output ~ 0
 BAT_PROBE
